File: PCB/_autosave-shield_led.kicad_pcb (KiCad board)
At the start: 2 copper layers, 5 parts

Commit message: Réorganisation des dossiers dans PCB et ajout du CI régulateur de tension
Parts:
- removed D1: LED, LED-8MM
- removed LDR1: PHOTORESISTANCE, Photoresistance
- removed R1, R2: R, R4
- removed SHIELD1: ARDUINO_SHIELD, ARDUINO_SHIELD
Routing:
- net N-000001: track 73.1 -> 0.00 mm
- net N-000005: track 35.4 -> 0.00 mm
- net N-000002: track 17.8 -> 0.00 mm
- net N-000003: track 8.04 -> 0.00 mm
- removed copper zone on B.Cu, net N-000004
