File: PCB/Version antérieure/shield_led.kicad_pcb (KiCad board)
At the start: 2 copper layers, 5 parts

Commit message: Réorganisation des dossiers dans PCB et ajout du CI régulateur de tension
Connections:
- SHIELD1 pad 9: (no net) -> N-000005
Routing:
- added copper zone on B.Cu, net N-000004
- removed copper zone on B.Cu, net N-000007
Changed lines of the file:
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@@
   (general
     (links 7)
-    (no_connects 0)
+    (no_connects 2)
     (area 181.7116 86.050001 254.379999 167.199733)
     (thickness 1.6)
@@
     (zones 0)
     (modules 5)
-    (nets 6)
+    (nets 7)
   )
   (page A3)
@@
   (net 2 N-000002)
   (net 3 N-000003)
-  (net 4 N-000004)
-  (net 5 N-000005)
+  (net 4 N-000005)
+  (net 5 N-000006)
+  (net 6 N-000007)
   (net_class Default "Ceci est la Netclass par défaut"
     (clearance 0.254)
@@
     (add_net N-000002)
     (add_net N-000003)
-    (add_net N-000004)
     (add_net N-000005)
+    (add_net N-000006)
+    (add_net N-000007)
   )
   (module R4 (layer Dessus.Cu)
@@
     (pad 2 thru_hole circle (at 5.08 0) (size 1.524 1.524) (drill 0.8128)
       (layers *.Cu *.Mask Dessus.SilkS)
-      (net 5 N-000005)
+      (net 5 N-000006)
     )
     (model discret/resistor.wrl
@@
     (pad 1 thru_hole circle (at -5.08 0) (size 1.524 1.524) (drill 0.8128)
       (layers *.Cu *.Mask Dessus.SilkS)
+      (net 2 N-000002)
+    )
+    (pad 2 thru_hole circle (at 5.08 0) (size 1.524 1.524) (drill 0.8128)
+      (layers *.Cu *.Mask Dessus.SilkS)
       (net 3 N-000003)
-    )
-    (pad 2 thru_hole circle (at 5.08 0) (size 1.524 1.524) (drill 0.8128)
-      (layers *.Cu *.Mask Dessus.SilkS)
-      (net 2 N-000002)
     )
     (model discret/resistor.wrl
@@
     (pad 1 thru_hole circle (at -4.89 -3.81) (size 1.5 1.5) (drill 0.69)
       (layers *.Cu *.Mask Dessus.SilkS)
-      (net 5 N-000005)
+      (net 5 N-000006)
     )
     (pad 2 thru_hole circle (at 4.89 -3.81) (size 1.5 1.5) (drill 0.69)
       (layers *.Cu *.Mask Dessus.SilkS)
-      (net 4 N-000004)
+      (net 6 N-000007)
     )
   )
@@
     (pad 1 thru_hole circle (at -1.27 0) (size 1.6764 1.6764) (drill 0.8128)
       (layers *.Cu *.Mask Dessus.SilkS)
-      (net 2 N-000002)
+      (net 3 N-000003)
     )
     (pad 2 thru_hole circle (at 1.27 0) (size 1.6764 1.6764) (drill 0.8128)
       (layers *.Cu *.Mask Dessus.SilkS)
-      (net 4 N-000004)
+      (net 6 N-000007)
     )
   )
@@
     (pad AD5 thru_hole oval (at 63.5 -2.54 180) (size 2.54 1.524) (drill 0.8128)
       (layers *.Cu *.Mask Dessus.SilkS)
-      (net 5 N-000005)
+      (net 5 N-000006)
     )
     (pad AD4 thru_hole oval (at 60.96 -2.54 180) (size 2.54 1.524) (drill 0.8128)
@@
     (pad GND1 thru_hole oval (at 40.64 -2.54 180) (size 2.54 1.524) (drill 0.8128)
       (layers *.Cu *.Mask Dessus.SilkS)
-      (net 4 N-000004)
+      (net 6 N-000007)
     )
     (pad 3V3 thru_hole oval (at 35.56 -2.54 180) (size 2.54 1.524) (drill 0.8128)
@@
     (pad 9 thru_hole oval (at 39.116 -50.8 180) (size 2.54 1.524) (drill 0.8128)
       (layers *.Cu *.Mask Dessus.SilkS)
+      (net 4 N-000005)
     )
     (pad 10 thru_hole oval (at 36.576 -50.8 180) (size 2.54 1.524) (drill 0.8128)
@@
     (pad 13 thru_hole oval (at 28.956 -50.8 180) (size 2.54 1.524) (drill 0.8128)
       (layers *.Cu *.Mask Dessus.SilkS)
-      (net 3 N-000003)
+      (net 2 N-000002)
     )
     (pad GND3 thru_hole oval (at 26.416 -50.8 180) (size 2.54 1.524) (drill 0.8128)
@@
   (segment (start 196.85 113.03) (end 220.98 113.03) (width 0.254) (layer Dessous.Cu) (net 1))
   (segment (start 195.58 111.76) (end 196.85 113.03) (width 0.254) (layer Dessous.Cu) (net 1))
-  (segment (start 207.01 137.16) (end 224.79 137.16) (width 0.254) (layer Dessous.Cu) (net 2))
-  (segment (start 189.23 136.144) (end 195.834 136.144) (width 0.254) (layer Dessous.Cu) (net 3))
-  (segment (start 195.834 136.144) (end 196.85 137.16) (width 0.254) (layer Dessous.Cu) (net 3))
+  (segment (start 189.23 136.144) (end 195.834 136.144) (width 0.254) (layer Dessous.Cu) (net 2))
+  (segment (start 195.834 136.144) (end 196.85 137.16) (width 0.254) (layer Dessous.Cu) (net 2))
+  (segment (start 207.01 137.16) (end 224.79 137.16) (width 0.254) (layer Dessous.Cu) (net 3))
   (segment (start 237.49 101.6) (end 226.25 101.6) (width 0.254) (layer Dessous.Cu) (net 5))
   (segment (start 226.25 101.6) (end 218.63 109.22) (width 0.254) (layer Dessous.Cu) (net 5))
   (segment (start 218.63 109.22) (end 207.01 109.22) (width 0.254) (layer Dessous.Cu) (net 5))
   (segment (start 207.01 109.22) (end 205.74 107.95) (width 0.254) (layer Dessous.Cu) (net 5))
-  (zone (net 4) (net_name N-000004) (layer Dessous.Cu) (hatch edge 0.508)
+  (zone (net -1) (net_name N-000004) (layer Dessous.Cu) (hatch edge 0.508)
     (connect_pads (clearance 0.508))
     (min_thickness 0.254)
