File: PCB/Régulateur/shield_7805.kicad_pcb (KiCad board)
At the start: 2 copper layers, 3 parts, among them P1 CONN_2, P2 CONN_4, U1 7805

Commit message: Version finale partie elec (Shield LDR & CI Regulateur)
Parts:
- moved P1 43.4 mm to (186.7, 160.0)
- moved P2 43.4 mm to (201.9, 160.0)
- moved U1 43.4 mm to (191.8, 143.5)
Routing:
- net N-000001: track 32.8 -> 0.00 mm
- net N-000002: track 27.0 -> 27.7 mm
- added copper zone on B.Cu, net N-000001
Other:
- net class Default: trace_width 0.254 -> 0.5
- board text added: "ASI 3"
Changed lines of the file:
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@@
     (links 6)
     (no_connects 0)
-    (area 223.469999 103.830001 263.269999 149.910001)
+    (area 176.479999 113.990001 239.139999 174.040001)
     (thickness 1.6)
-    (drawings 6)
-    (tracks 18)
+    (drawings 11)
+    (tracks 7)
     (zones 0)
     (modules 3)
@@
   )
   (setup
-    (last_trace_width 0.254)
+    (last_trace_width 0.5)
     (trace_clearance 0.254)
     (zone_clearance 0.508)
@@
   (net_class Default "Ceci est la Netclass par défaut"
     (clearance 0.254)
-    (trace_width 0.254)
+    (trace_width 0.5)
     (via_dia 0.889)
     (via_drill 0.635)
@@
   )
   (module PIN_ARRAY_4x1 (layer Dessus.Cu)
-    (at 242.57 144.78 180)
+    (at 201.93 160.02 180)
     (descr "Double rangee de contacts 2 x 5 pins")
     (tags CONN)
@@
   )
   (module PIN_ARRAY_2X1 (layer Dessus.Cu)
-    (at 227.33 144.78)
+    (at 186.69 160.02)
     (descr "Connecteurs 2 pins")
     (tags "CONN DEV")
@@
   )
   (module 7805 (layer Dessus.Cu)
-    (at 232.41 128.27)
+    (at 191.77 143.51)
     (fp_text reference U1 (at 0 -1.27) (layer Dessus.SilkS)
       (effects (font (size 1 1) (thickness 0.15)))
@@
     )
   )
-  (dimension 38.1 (width 0.3) (layer Contours.Ci)
-    (gr_text "38,100 mm" (at 256.619999 130.81 270) (layer Contours.Ci)
+  (dimension 49.53 (width 0.3) (layer Contours.Ci)
+    (gr_text "49,530 mm" (at 232.489999 149.225 270) (layer Contours.Ci)
       (effects (font (size 1.5 1.5) (thickness 0.3)))
     )
-    (feature1 (pts (xy 252.73 149.86) (xy 257.969999 149.86)))
-    (feature2 (pts (xy 252.73 111.76) (xy 257.969999 111.76)))
-    (crossbar (pts (xy 255.269999 111.76) (xy 255.269999 149.86)))
-    (arrow1a (pts (xy 255.269999 149.86) (xy 254.683579 148.733497)))
-    (arrow1b (pts (xy 255.269999 149.86) (xy 255.856419 148.733497)))
-    (arrow2a (pts (xy 255.269999 111.76) (xy 254.683579 112.886503)))
-    (arrow2b (pts (xy 255.269999 111.76) (xy 255.856419 112.886503)))
-  )
-  (dimension 26.67 (width 0.3) (layer Contours.Ci)
-    (gr_text "26,670 mm" (at 236.855 105.330001) (layer Contours.Ci)
+    (feature1 (pts (xy 223.52 173.99) (xy 233.839999 173.99)))
+    (feature2 (pts (xy 223.52 124.46) (xy 233.839999 124.46)))
+    (crossbar (pts (xy 231.139999 124.46) (xy 231.139999 173.99)))
+    (arrow1a (pts (xy 231.139999 173.99) (xy 230.553579 172.863497)))
+    (arrow1b (pts (xy 231.139999 173.99) (xy 231.726419 172.863497)))
+    (arrow2a (pts (xy 231.139999 124.46) (xy 230.553579 125.586503)))
+    (arrow2b (pts (xy 231.139999 124.46) (xy 231.726419 125.586503)))
+  )
+  (gr_line (start 217.17 173.99) (end 217.17 162.56) (angle 90) (layer Contours.Ci) (width 0.1))
+  (gr_line (start 176.53 173.99) (end 217.17 173.99) (angle 90) (layer Contours.Ci) (width 0.1))
+  (gr_line (start 176.53 162.56) (end 176.53 173.99) (angle 90) (layer Contours.Ci) (width 0.1))
+  (gr_text "ASI 3" (at 207.01 135.89) (layer Dessous.Cu)
+    (effects (font (size 3 3) (thickness 0.3)) (justify mirror))
+  )
+  (dimension 41.91 (width 0.3) (layer Contours.Ci)
+    (gr_text "41,910 mm" (at 197.485 115.490001) (layer Contours.Ci)
       (effects (font (size 1.5 1.5) (thickness 0.3)))
     )
-    (feature1 (pts (xy 250.19 109.22) (xy 250.19 103.980001)))
-    (feature2 (pts (xy 223.52 109.22) (xy 223.52 103.980001)))
-    (crossbar (pts (xy 223.52 106.680001) (xy 250.19 106.680001)))
-    (arrow1a (pts (xy 250.19 106.680001) (xy 249.063497 107.266421)))
-    (arrow1b (pts (xy 250.19 106.680001) (xy 249.063497 106.093581)))
-    (arrow2a (pts (xy 223.52 106.680001) (xy 224.646503 107.266421)))
-    (arrow2b (pts (xy 223.52 106.680001) (xy 224.646503 106.093581)))
-  )
-  (gr_line (start 223.52 111.76) (end 250.19 111.76) (angle 90) (layer Contours.Ci) (width 0.1))
-  (gr_line (start 223.52 149.86) (end 223.52 111.76) (angle 90) (layer Contours.Ci) (width 0.1))
-  (gr_line (start 250.19 149.86) (end 223.52 149.86) (angle 90) (layer Contours.Ci) (width 0.1))
-  (gr_line (start 250.19 111.76) (end 250.19 149.86) (angle 90) (layer Contours.Ci) (width 0.1))
-  (segment (start 238.76 138.43) (end 238.76 144.78) (width 0.254) (layer Dessous.Cu) (net 1) (status 800000))
-  (segment (start 232.41 138.43) (end 238.76 138.43) (width 0.254) (layer Dessous.Cu) (net 1))
-  (segment (start 238.76 138.43) (end 240.03 138.43) (width 0.254) (layer Dessous.Cu) (net 1))
-  (segment (start 241.3 139.7) (end 241.3 144.78) (width 0.254) (layer Dessous.Cu) (net 1) (status 800000))
-  (segment (start 240.03 138.43) (end 241.3 139.7) (width 0.254) (layer Dessous.Cu) (net 1))
-  (segment (start 232.41 135.89) (end 232.41 138.43) (width 0.254) (layer Dessous.Cu) (net 1) (status 400000))
-  (segment (start 228.6 139.7) (end 228.6 144.78) (width 0.254) (layer Dessous.Cu) (net 1) (status 800000))
-  (segment (start 229.87 138.43) (end 228.6 139.7) (width 0.254) (layer Dessous.Cu) (net 1))
-  (segment (start 232.41 138.43) (end 229.87 138.43) (width 0.254) (layer Dessous.Cu) (net 1))
-  (segment (start 245.11 137.16) (end 243.84 138.43) (width 0.254) (layer Dessous.Cu) (net 2))
-  (segment (start 243.84 138.43) (end 243.84 144.78) (width 0.254) (layer Dessous.Cu) (net 2) (status 800000))
-  (segment (start 234.95 135.89) (end 243.84 135.89) (width 0.254) (layer Dessous.Cu) (net 2) (status 400000))
-  (segment (start 243.84 135.89) (end 245.11 137.16) (width 0.254) (layer Dessous.Cu) (net 2))
-  (segment (start 245.11 137.16) (end 246.38 138.43) (width 0.254) (layer Dessous.Cu) (net 2))
-  (segment (start 246.38 138.43) (end 246.38 144.78) (width 0.254) (layer Dessous.Cu) (net 2))
-  (segment (start 229.87 135.89) (end 227.33 135.89) (width 0.254) (layer Dessous.Cu) (net 3) (status 400000))
-  (segment (start 226.06 137.16) (end 226.06 144.78) (width 0.254) (layer Dessous.Cu) (net 3) (status 800000))
-  (segment (start 227.33 135.89) (end 226.06 137.16) (width 0.254) (layer Dessous.Cu) (net 3))
+    (feature1 (pts (xy 218.44 118.11) (xy 218.44 114.140001)))
+    (feature2 (pts (xy 176.53 118.11) (xy 176.53 114.140001)))
+    (crossbar (pts (xy 176.53 116.840001) (xy 218.44 116.840001)))
+    (arrow1a (pts (xy 218.44 116.840001) (xy 217.313497 117.426421)))
+    (arrow1b (pts (xy 218.44 116.840001) (xy 217.313497 116.253581)))
+    (arrow2a (pts (xy 176.53 116.840001) (xy 177.656503 117.426421)))
+    (arrow2b (pts (xy 176.53 116.840001) (xy 177.656503 116.253581)))
+  )
+  (gr_line (start 217.17 124.46) (end 217.17 162.56) (angle 90) (layer Contours.Ci) (width 0.1))
+  (gr_line (start 213.36 124.46) (end 217.17 124.46) (angle 90) (layer Contours.Ci) (width 0.1))
+  (gr_line (start 203.2 124.46) (end 213.36 124.46) (angle 90) (layer Contours.Ci) (width 0.1))
+  (gr_line (start 176.53 124.46) (end 203.2 124.46) (angle 90) (layer Contours.Ci) (width 0.1))
+  (gr_line (start 176.53 162.56) (end 176.53 124.46) (angle 90) (layer Contours.Ci) (width 0.1))
+  (segment (start 203.2 160.02) (end 203.2 151.13) (width 0.5) (layer Dessous.Cu) (net 2) (status 400000))
+  (segment (start 194.31 151.13) (end 203.2 151.13) (width 0.5) (layer Dessous.Cu) (net 2) (status 400000))
+  (segment (start 205.74 153.67) (end 205.74 160.02) (width 0.5) (layer Dessous.Cu) (net 2) (status 800000))
+  (segment (start 203.2 151.13) (end 205.74 153.67) (width 0.5) (layer Dessous.Cu) (net 2))
+  (segment (start 189.23 151.13) (end 186.69 151.13) (width 0.5) (layer Dessous.Cu) (net 3) (status 400000))
+  (segment (start 185.42 152.4) (end 185.42 160.02) (width 0.5) (layer Dessous.Cu) (net 3) (status 800000))
+  (segment (start 186.69 151.13) (end 185.42 152.4) (width 0.5) (layer Dessous.Cu) (net 3))
+  (zone (net 1) (net_name N-000001) (layer Dessous.Cu) (hatch edge 0.508)
+    (connect_pads (clearance 0.508))
+    (min_thickness 0.254)
+    (fill (arc_segments 16) (thermal_gap 0.508) (thermal_bridge_width 0.508))
+    (polygon
+      (pts
+        (xy 217.17 173.99) (xy 176.53 173.99) (xy 176.53 124.46) (xy 217.17 124.46)
+      )
+    )
+  )
 )
