File: PCB/Shield-LDR/shield_LDR.sch (KiCad schematic (older format))
At the start: 7 parts

Commit message: Version finale partie elec (Shield LDR & CI Regulateur)
Connections:
- net at SHIELD1.9: no longer R3.1
- net at SHIELD1.AD1: now also R3.1
Changed lines of the file:
@@
-EESchema Schematic File Version 2  date 29/10/2013 15:11:44
+EESchema Schematic File Version 2  date 15/11/2013 21:16:23
 LIBS:power
 LIBS:device
@@
 Sheet 1 1
 Title "noname.sch"
-Date "29 oct 2013"
+Date "15 nov 2013"
 Rev ""
 Comp ""
@@
 $EndComp
 Wire Wire Line
-	5750 3400 6450 3400
-Wire Wire Line
-	6450 3400 6450 5500
-Wire Wire Line
 	6950 5500 7500 5500
 Wire Wire Line
@@
 	8350 5500 8350 4700
 Connection ~ 8350 4700
+Wire Wire Line
+	3850 4000 3500 4000
+Wire Wire Line
+	3500 4000 3500 5500
+Wire Wire Line
+	3500 5500 6450 5500
 $EndSCHEMATC
