File: PCB/Shield-LDR/shield_LDRv2.kicad_pcb (KiCad board)
At the start: 2 copper layers, 7 parts

Commit message: Version finale partie elec (Shield LDR & CI Regulateur)
Connections:
- SHIELD1 pad 9: N-000005 -> (no net)
- SHIELD1 pad AD1: (no net) -> N-000005
Routing:
- net N-000005: track 9.52 -> 46.9 mm
- net N-000002: track 49.0 -> 70.8 mm
Other:
- net class Default: trace_width 0.254 -> 0.5
- board text added: "ASI 3"
Changed lines of the file:
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@@
     (area 128.3716 88.590001 203.579999 168.469733)
     (thickness 1.6)
-    (drawings 11)
-    (tracks 19)
+    (drawings 12)
+    (tracks 23)
     (zones 0)
     (modules 7)
@@
   )
   (setup
-    (last_trace_width 0.254)
+    (last_trace_width 0.5)
     (trace_clearance 0.254)
     (zone_clearance 0.508)
@@
   (net_class Default "Ceci est la Netclass par défaut"
     (clearance 0.254)
-    (trace_width 0.254)
+    (trace_width 0.5)
     (via_dia 0.889)
     (via_drill 0.635)
@@
     (tags R)
     (autoplace_cost180 10)
-    (fp_text reference R1 (at 0 0) (layer Dessus.SilkS)
+    (fp_text reference R1 (at 0 2.54) (layer Dessus.SilkS)
       (effects (font (size 1.397 1.27) (thickness 0.2032)))
     )
@@
     (pad 1 thru_hole circle (at -5.08 0) (size 1.524 1.524) (drill 0.8128)
       (layers *.Cu *.Mask Dessus.SilkS)
-      (net 1 N-000001)
+      (net 2 N-000002)
     )
     (pad 2 thru_hole circle (at 5.08 0) (size 1.524 1.524) (drill 0.8128)
       (layers *.Cu *.Mask Dessus.SilkS)
-      (net 6 N-000006)
+      (net 7 N-000007)
     )
     (model discret/resistor.wrl
@@
     (tags R)
     (autoplace_cost180 10)
-    (fp_text reference R2 (at 0 0) (layer Dessus.SilkS)
+    (fp_text reference R2 (at 0 2.54) (layer Dessus.SilkS)
       (effects (font (size 1.397 1.27) (thickness 0.2032)))
     )
@@
     (pad 1 thru_hole circle (at -5.08 0) (size 1.524 1.524) (drill 0.8128)
       (layers *.Cu *.Mask Dessus.SilkS)
-      (net 2 N-000002)
+      (net 3 N-000003)
     )
     (pad 2 thru_hole circle (at 5.08 0) (size 1.524 1.524) (drill 0.8128)
       (layers *.Cu *.Mask Dessus.SilkS)
-      (net 3 N-000003)
+      (net 6 N-000006)
     )
     (model discret/resistor.wrl
@@
     (tags R)
     (autoplace_cost180 10)
-    (fp_text reference R3 (at 0 0) (layer Dessus.SilkS)
+    (fp_text reference R3 (at 0 2.54) (layer Dessus.SilkS)
       (effects (font (size 1.397 1.27) (thickness 0.2032)))
     )
@@
     (pad 1 thru_hole circle (at -4.89 -3.81) (size 1 1) (drill 0.69)
       (layers *.Cu *.Mask Dessus.SilkS)
-      (net 6 N-000006)
+      (net 7 N-000007)
     )
     (pad 2 thru_hole circle (at 4.89 -3.81) (size 1 1) (drill 0.69)
       (layers *.Cu *.Mask Dessus.SilkS)
-      (net 7 N-000007)
+      (net 1 N-000001)
     )
   )
@@
     (pad 1 thru_hole circle (at -1.27 0) (size 1.6764 1.6764) (drill 0.8128)
       (layers *.Cu *.Mask Dessus.SilkS)
-      (net 3 N-000003)
+      (net 6 N-000006)
     )
     (pad 2 thru_hole circle (at 1.27 0) (size 1.6764 1.6764) (drill 0.8128)
       (layers *.Cu *.Mask Dessus.SilkS)
-      (net 7 N-000007)
+      (net 1 N-000001)
     )
     (model discret/leds/led5_vertical_verde.wrl
@@
     (pad 2 thru_hole circle (at 1.27 0) (size 1.6764 1.6764) (drill 0.8128)
       (layers *.Cu *.Mask Dessus.SilkS)
-      (net 7 N-000007)
+      (net 1 N-000001)
     )
     (model discret/leds/led5_vertical_verde.wrl
@@
     (pad AD5 thru_hole oval (at 63.5 -2.54 180) (size 2.54 1.524) (drill 0.8128)
       (layers *.Cu *.Mask Dessus.SilkS)
-      (net 6 N-000006)
+      (net 7 N-000007)
     )
     (pad AD4 thru_hole oval (at 60.96 -2.54 180) (size 2.54 1.524) (drill 0.8128)
@@
     (pad AD1 thru_hole oval (at 53.34 -2.54 180) (size 2.54 1.524) (drill 0.8128)
       (layers *.Cu *.Mask Dessus.SilkS)
+      (net 5 N-000005)
     )
     (pad AD2 thru_hole oval (at 55.88 -2.54 180) (size 2.54 1.524) (drill 0.8128)
@@
     (pad GND1 thru_hole oval (at 40.64 -2.54 180) (size 2.54 1.524) (drill 0.8128)
       (layers *.Cu *.Mask Dessus.SilkS)
-      (net 7 N-000007)
+      (net 1 N-000001)
     )
     (pad 3V3 thru_hole oval (at 35.56 -2.54 180) (size 2.54 1.524) (drill 0.8128)
@@
     (pad 9 thru_hole oval (at 39.116 -50.8 180) (size 2.54 1.524) (drill 0.8128)
       (layers *.Cu *.Mask Dessus.SilkS)
-      (net 5 N-000005)
     )
     (pad 10 thru_hole oval (at 36.576 -50.8 180) (size 2.54 1.524) (drill 0.8128)
@@
     (pad 13 thru_hole oval (at 28.956 -50.8 180) (size 2.54 1.524) (drill 0.8128)
       (layers *.Cu *.Mask Dessus.SilkS)
+      (net 3 N-000003)
+    )
+    (pad GND3 thru_hole oval (at 26.416 -50.8 180) (size 2.54 1.524) (drill 0.8128)
+      (layers *.Cu *.Mask Dessus.SilkS)
+    )
+    (pad AREF thru_hole oval (at 23.876 -50.8 180) (size 2.54 1.524) (drill 0.8128)
+      (layers *.Cu *.Mask Dessus.SilkS)
+    )
+    (pad 5V thru_hole oval (at 38.1 -2.54 180) (size 2.54 1.524) (drill 0.8128)
+      (layers *.Cu *.Mask Dessus.SilkS)
       (net 2 N-000002)
     )
-    (pad GND3 thru_hole oval (at 26.416 -50.8 180) (size 2.54 1.524) (drill 0.8128)
-      (layers *.Cu *.Mask Dessus.SilkS)
-    )
-    (pad AREF thru_hole oval (at 23.876 -50.8 180) (size 2.54 1.524) (drill 0.8128)
-      (layers *.Cu *.Mask Dessus.SilkS)
-    )
-    (pad 5V thru_hole oval (at 38.1 -2.54 180) (size 2.54 1.524) (drill 0.8128)
-      (layers *.Cu *.Mask Dessus.SilkS)
-      (net 1 N-000001)
-    )
     (pad "" thru_hole circle (at 66.04 -7.62 180) (size 3.937 3.937) (drill 3.175)
       (layers *.Cu *.Mask Dessus.SilkS)
@@
       (layers *.Cu *.Mask Dessus.SilkS)
     )
+  )
+  (gr_text "ASI 3" (at 160.02 148.59) (layer Dessous.Cu)
+    (effects (font (size 4 4) (thickness 0.3)) (justify mirror))
   )
   (dimension 68.58 (width 0.3) (layer Contours.Ci)
@@
   (gr_line (start 146.05 100.33) (end 148.59 97.79) (angle 90) (layer Contours.Ci) (width 0.15))
   (gr_line (start 134.62 100.33) (end 146.05 100.33) (angle 90) (layer Contours.Ci) (width 0.15))
-  (segment (start 146.05 109.22) (end 146.05 114.3) (width 0.254) (layer Dessous.Cu) (net 1))
-  (segment (start 179.07 128.27) (end 184.15 128.27) (width 0.254) (layer Dessous.Cu) (net 1))
-  (segment (start 171.45 120.65) (end 179.07 128.27) (width 0.254) (layer Dessous.Cu) (net 1))
-  (segment (start 152.4 120.65) (end 171.45 120.65) (width 0.254) (layer Dessous.Cu) (net 1))
-  (segment (start 146.05 114.3) (end 152.4 120.65) (width 0.254) (layer Dessous.Cu) (net 1))
-  (segment (start 144.78 137.16) (end 136.144 137.16) (width 0.254) (layer Dessous.Cu) (net 2))
-  (segment (start 136.144 137.16) (end 135.89 137.414) (width 0.254) (layer Dessous.Cu) (net 2))
-  (segment (start 154.94 137.16) (end 167.64 137.16) (width 0.254) (layer Dessous.Cu) (net 3))
-  (segment (start 154.94 125.73) (end 167.64 125.73) (width 0.254) (layer Dessous.Cu) (net 4))
-  (segment (start 144.78 125.73) (end 140.97 125.73) (width 0.254) (layer Dessous.Cu) (net 5))
-  (segment (start 139.446 127.254) (end 135.89 127.254) (width 0.254) (layer Dessous.Cu) (net 5))
-  (segment (start 140.97 125.73) (end 139.446 127.254) (width 0.254) (layer Dessous.Cu) (net 5))
-  (segment (start 164.02 110.49) (end 167.64 110.49) (width 0.254) (layer Dessous.Cu) (net 6))
-  (segment (start 180.34 102.87) (end 184.15 102.87) (width 0.254) (layer Dessous.Cu) (net 6))
-  (segment (start 179.07 104.14) (end 180.34 102.87) (width 0.254) (layer Dessous.Cu) (net 6))
-  (segment (start 173.99 104.14) (end 179.07 104.14) (width 0.254) (layer Dessous.Cu) (net 6))
-  (segment (start 167.64 110.49) (end 173.99 104.14) (width 0.254) (layer Dessous.Cu) (net 6))
-  (segment (start 156.21 109.22) (end 162.75 109.22) (width 0.254) (layer Dessous.Cu) (net 6))
-  (segment (start 162.75 109.22) (end 164.02 110.49) (width 0.254) (layer Dessous.Cu) (net 6))
-  (zone (net 7) (net_name N-000007) (layer Dessous.Cu) (hatch edge 0.508)
+  (segment (start 146.05 109.22) (end 143.51 109.22) (width 0.5) (layer Dessous.Cu) (net 2))
+  (segment (start 143.51 109.22) (end 139.7 113.03) (width 0.5) (layer Dessous.Cu) (net 2))
+  (segment (start 139.7 113.03) (end 139.7 128.27) (width 0.5) (layer Dessous.Cu) (net 2))
+  (segment (start 139.7 128.27) (end 143.51 132.08) (width 0.5) (layer Dessous.Cu) (net 2))
+  (segment (start 143.51 132.08) (end 175.26 132.08) (width 0.5) (layer Dessous.Cu) (net 2))
+  (segment (start 175.26 132.08) (end 179.07 128.27) (width 0.5) (layer Dessous.Cu) (net 2))
+  (segment (start 179.07 128.27) (end 184.15 128.27) (width 0.5) (layer Dessous.Cu) (net 2))
+  (segment (start 144.78 137.16) (end 136.144 137.16) (width 0.5) (layer Dessous.Cu) (net 3))
+  (segment (start 136.144 137.16) (end 135.89 137.414) (width 0.5) (layer Dessous.Cu) (net 3))
+  (segment (start 154.94 125.73) (end 167.64 125.73) (width 0.5) (layer Dessous.Cu) (net 4))
+  (segment (start 144.78 125.73) (end 144.78 121.92) (width 0.5) (layer Dessous.Cu) (net 5))
+  (segment (start 144.78 121.92) (end 149.86 116.84) (width 0.5) (layer Dessous.Cu) (net 5))
+  (segment (start 149.86 116.84) (end 173.99 116.84) (width 0.5) (layer Dessous.Cu) (net 5))
+  (segment (start 173.99 116.84) (end 177.8 113.03) (width 0.5) (layer Dessous.Cu) (net 5))
+  (segment (start 177.8 113.03) (end 184.15 113.03) (width 0.5) (layer Dessous.Cu) (net 5))
+  (segment (start 154.94 137.16) (end 167.64 137.16) (width 0.5) (layer Dessous.Cu) (net 6))
+  (segment (start 164.02 110.49) (end 167.64 110.49) (width 0.5) (layer Dessous.Cu) (net 7))
+  (segment (start 167.64 110.49) (end 173.99 104.14) (width 0.5) (layer Dessous.Cu) (net 7))
+  (segment (start 173.99 104.14) (end 179.07 104.14) (width 0.5) (layer Dessous.Cu) (net 7))
+  (segment (start 179.07 104.14) (end 180.34 102.87) (width 0.5) (layer Dessous.Cu) (net 7))
+  (segment (start 180.34 102.87) (end 184.15 102.87) (width 0.5) (layer Dessous.Cu) (net 7))
+  (segment (start 156.21 109.22) (end 162.75 109.22) (width 0.5) (layer Dessous.Cu) (net 7))
+  (segment (start 162.75 109.22) (end 164.02 110.49) (width 0.5) (layer Dessous.Cu) (net 7))
+  (zone (net 1) (net_name N-000001) (layer Dessous.Cu) (hatch edge 0.508)
     (connect_pads (clearance 0.508))
     (min_thickness 0.254)
